File: watch_hw/watch.kicad_pcb (KiCad board)
At the start: 6 copper layers, 36.4 x 38.8 mm, 55 parts, among them J1 USB_B_Micro, J3 Conn_ARM_SWD_TagConnect_TC203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, SW1 TL6340AF160Q, SW2 TL6340AF160Q, U1 STM32WB55CGUx, U2 nPM1100-QDAA, U3 MAX17048G+, U4 BMA456, U5 MAXM86161EFD+T, X1 NX2016SA-32M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

Commit message: finish routing, need to fix DRC
Parts:
- moved R4 17.4 mm to (143.4, 110.0)
- moved R3 17.2 mm to (143.4, 111.2)
- moved C5 1.40 mm to (144.2, 112.4), turned to 180 degrees
- moved R8 1.12 mm to (164.2, 106.0)
- moved C12 0.90 mm to (149.6, 114.4)
- moved R1 0.85 mm to (150.9, 114.4)
- moved C7 0.85 mm to (152.9, 113.6)
- moved C8 0.85 mm to (152.9, 115.1)
- moved C16 0.81 mm to (151.5, 104.8)
- moved R2 0.70 mm to (150.2, 117.2)
- moved C15 0.60 mm to (146.1, 100.0)
- moved C10 0.41 mm to (143.9, 107.1), turned to 180 degrees
- moved C25 0.10 mm to (156.1, 100.8)
- moved R7 0.10 mm to (164.0, 94.2)
- moved C2 0.08 mm to (155.7, 105.5)
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Connections:
- U1 pad 11: unconnected-(U1-PA2-Pad11) -> /BTN0
- U1 pad 12: unconnected-(U1-PA3-Pad12) -> /BTN1
- U1 pad 42: unconnected-(U1-PA15-Pad42) -> /Power/BAT_ERR
- U1 pad 43: unconnected-(U1-PB3-Pad43) -> /Power/BAT_CHG
- U1 pad 44: unconnected-(U1-PB4-Pad44) -> /Power/~{BAT_ALRT}
- U1 pad 45: unconnected-(U1-PB5-Pad45) -> /Sensors/ACC_INT
- U1 pad 46: unconnected-(U1-PB6-Pad46) -> /SCL
- U1 pad 47: unconnected-(U1-PB7-Pad47) -> /SDA
- U2 pad 19: /USB_D_N -> GND
- U2 pad 20: /USB_D_P -> unconnected-(U2-D+-Pad20)
Routing:
- net /SDA: track 15.5 -> 55.2 mm, vias 2 -> 4
- net /SCL: track 12.0 -> 51.3 mm, vias 1 -> 3
- net /Power/~{BAT_ALRT}: track 0.00 -> 31.3 mm, vias 0 -> 2
- net /Power/BAT_CHG: track 0.00 -> 26.9 mm, vias 0 -> 2
- net /Sensors/ACC_INT: track 0.00 -> 26.6 mm, vias 0 -> 2
- net /Power/BAT_ERR: track 0.00 -> 25.2 mm, vias 0 -> 2
- net VDD: track 45.2 -> 70.4 mm, vias 0 -> 19
- net /BTN0: track 1.90 -> 26.2 mm, vias 0 -> 2
- net /BTN1: track 5.71 -> 22.8 mm, vias 0 -> 2
- net /SoC/NRST: track 3.44 -> 18.1 mm, vias 0 -> 2
- net /USB_D_P: track 0.00 -> 12.7 mm, vias 0 -> 2
- net /USB_D_N: track 0.00 -> 12.7 mm, vias 0 -> 2
- net /SoC/SWDIO: track 0.00 -> 6.56 mm
- net /Power/VSYS: track 17.4 -> 11.5 mm
- net /Power/VBAT: track 18.5 -> 23.4 mm
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- added copper zone on In3.Cu, net /Power/VSYS
- added copper zone on B.Cu, net GND
- added copper zone on F.Cu, net GND
- added copper zone on In2.Cu, net VDD
- added copper zone on In3.Cu, net VDD

Commit message: pass DRC
Parts:
- L1: footprint Inductor_SMD:L_0805_2012Metric_Pad1.15x1.40mm_HandSolder -> Inductor_SMD:L_0805_2012Metric_Pad1.05x1.20mm_HandSolder
- moved R8 1.43 mm to (163.9, 107.4)
- moved SW1 1.00 mm to (166.9, 95.5)
- moved SW2 1.00 mm to (166.9, 104.5)
- moved R7 0.63 mm to (163.4, 94.4)
- renumbered REF** to DISP
Routing:
- net /BTN1: track 22.8 -> 23.8 mm
