File: watch_hw/display.kicad_sch (KiCad schematic)
At the start: 4 parts

Commit message: Finalize (?) part selection, start layout
Parts:
- renumbered C37 to C24, C38 to C25, C39 to C26
Changed lines of the file:
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@@
   (symbol (lib_id "power:GND") (at 114.3 118.11 0) (unit 1)
     (in_bom yes) (on_board yes) (dnp no) (fields_autoplaced)
-    (property "Reference" "#PWR085" (at 114.3 124.46 0)
+    (property "Reference" "#PWR064" (at 114.3 124.46 0)
       (effects (font (size 1.27 1.27)) hide)
     )
@@
       (project "watch"
         (path "/7f737de8-b7e5-4967-9e9f-b541c91fc2b3/2a2ea5a3-6605-4888-bae5-df756037ea07"
-          (reference "#PWR085") (unit 1)
+          (reference "#PWR064") (unit 1)
         )
       )
@@
   (symbol (lib_id "power:GND") (at 170.18 101.6 0) (unit 1)
     (in_bom yes) (on_board yes) (dnp no) (fields_autoplaced)
-    (property "Reference" "#PWR082" (at 170.18 107.95 0)
+    (property "Reference" "#PWR061" (at 170.18 107.95 0)
       (effects (font (size 1.27 1.27)) hide)
     )
@@
       (project "watch"
         (path "/7f737de8-b7e5-4967-9e9f-b541c91fc2b3/2a2ea5a3-6605-4888-bae5-df756037ea07"
-          (reference "#PWR082") (unit 1)
+          (reference "#PWR061") (unit 1)
         )
       )
@@
   (symbol (lib_id "power:VDD") (at 157.48 93.98 0) (unit 1)
     (in_bom yes) (on_board yes) (dnp no) (fields_autoplaced)
-    (property "Reference" "#PWR079" (at 157.48 97.79 0)
+    (property "Reference" "#PWR058" (at 157.48 97.79 0)
       (effects (font (size 1.27 1.27)) hide)
     )
@@
       (project "watch"
         (path "/7f737de8-b7e5-4967-9e9f-b541c91fc2b3/2a2ea5a3-6605-4888-bae5-df756037ea07"
-          (reference "#PWR079") (unit 1)
+          (reference "#PWR058") (unit 1)
         )
       )
@@
   (symbol (lib_id "power:GND") (at 83.82 105.41 0) (unit 1)
     (in_bom yes) (on_board yes) (dnp no) (fields_autoplaced)
-    (property "Reference" "#PWR083" (at 83.82 111.76 0)
+    (property "Reference" "#PWR062" (at 83.82 111.76 0)
       (effects (font (size 1.27 1.27)) hide)
     )
@@
       (project "watch"
         (path "/7f737de8-b7e5-4967-9e9f-b541c91fc2b3/2a2ea5a3-6605-4888-bae5-df756037ea07"
-          (reference "#PWR083") (unit 1)
+          (reference "#PWR062") (unit 1)
         )
       )
@@
   (symbol (lib_id "Device:C_Small") (at 83.82 101.6 0) (unit 1)
     (in_bom yes) (on_board yes) (dnp no)
-    (property "Reference" "C39" (at 81.28 100.33 0)
+    (property "Reference" "C26" (at 81.28 100.33 0)
       (effects (font (size 1.27 1.27)) (justify right))
     )
@@
       (project "watch"
         (path "/7f737de8-b7e5-4967-9e9f-b541c91fc2b3/2a2ea5a3-6605-4888-bae5-df756037ea07"
-          (reference "C39") (unit 1)
+          (reference "C26") (unit 1)
         )
       )
@@
   (symbol (lib_id "power:VDD") (at 114.3 74.93 0) (unit 1)
     (in_bom yes) (on_board yes) (dnp no) (fields_autoplaced)
-    (property "Reference" "#PWR077" (at 114.3 78.74 0)
+    (property "Reference" "#PWR056" (at 114.3 78.74 0)
       (effects (font (size 1.27 1.27)) hide)
     )
@@
       (project "watch"
         (path "/7f737de8-b7e5-4967-9e9f-b541c91fc2b3/2a2ea5a3-6605-4888-bae5-df756037ea07"
-          (reference "#PWR077") (unit 1)
+          (reference "#PWR056") (unit 1)
         )
       )
@@
   (symbol (lib_id "power:VDD") (at 170.18 93.98 0) (unit 1)
     (in_bom yes) (on_board yes) (dnp no) (fields_autoplaced)
-    (property "Reference" "#PWR080" (at 170.18 97.79 0)
+    (property "Reference" "#PWR059" (at 170.18 97.79 0)
       (effects (font (size 1.27 1.27)) hide)
     )
@@
       (project "watch"
         (path "/7f737de8-b7e5-4967-9e9f-b541c91fc2b3/2a2ea5a3-6605-4888-bae5-df756037ea07"
-          (reference "#PWR080") (unit 1)
+          (reference "#PWR059") (unit 1)
         )
       )
@@
   (symbol (lib_id "power:VDD") (at 109.22 74.93 0) (unit 1)
     (in_bom yes) (on_board yes) (dnp no) (fields_autoplaced)
-    (property "Reference" "#PWR076" (at 109.22 78.74 0)
+    (property "Reference" "#PWR055" (at 109.22 78.74 0)
       (effects (font (size 1.27 1.27)) hide)
     )
@@
       (project "watch"
         (path "/7f737de8-b7e5-4967-9e9f-b541c91fc2b3/2a2ea5a3-6605-4888-bae5-df756037ea07"
-          (reference "#PWR076") (unit 1)
+          (reference "#PWR055") (unit 1)
         )
       )
@@
   (symbol (lib_id "Device:C_Small") (at 157.48 97.79 0) (unit 1)
     (in_bom yes) (on_board yes) (dnp no) (fields_autoplaced)
-    (property "Reference" "C37" (at 160.02 96.5262 0)
+    (property "Reference" "C24" (at 160.02 96.5262 0)
       (effects (font (size 1.27 1.27)) (justify left))
     )
@@
       (project "watch"
         (path "/7f737de8-b7e5-4967-9e9f-b541c91fc2b3/2a2ea5a3-6605-4888-bae5-df756037ea07"
-          (reference "C37") (unit 1)
+          (reference "C24") (unit 1)
         )
       )
@@
   (symbol (lib_id "power:GND") (at 157.48 101.6 0) (unit 1)
     (in_bom yes) (on_board yes) (dnp no) (fields_autoplaced)
-    (property "Reference" "#PWR081" (at 157.48 107.95 0)
+    (property "Reference" "#PWR060" (at 157.48 107.95 0)
       (effects (font (size 1.27 1.27)) hide)
     )
@@
       (project "watch"
         (path "/7f737de8-b7e5-4967-9e9f-b541c91fc2b3/2a2ea5a3-6605-4888-bae5-df756037ea07"
-          (reference "#PWR081") (unit 1)
+          (reference "#PWR060") (unit 1)
         )
       )
@@
   (symbol (lib_id "Device:C_Small") (at 170.18 97.79 0) (unit 1)
     (in_bom yes) (on_board yes) (dnp no) (fields_autoplaced)
-    (property "Reference" "C38" (at 172.72 96.5262 0)
+    (property "Reference" "C25" (at 172.72 96.5262 0)
       (effects (font (size 1.27 1.27)) (justify left))
     )
@@
       (project "watch"
         (path "/7f737de8-b7e5-4967-9e9f-b541c91fc2b3/2a2ea5a3-6605-4888-bae5-df756037ea07"
-          (reference "C38") (unit 1)
+          (reference "C25") (unit 1)
         )
       )
@@
   (symbol (lib_id "power:GND") (at 109.22 118.11 0) (unit 1)
     (in_bom yes) (on_board yes) (dnp no) (fields_autoplaced)
-    (property "Reference" "#PWR084" (at 109.22 124.46 0)
+    (property "Reference" "#PWR063" (at 109.22 124.46 0)
       (effects (font (size 1.27 1.27)) hide)
     )
@@
       (project "watch"
         (path "/7f737de8-b7e5-4967-9e9f-b541c91fc2b3/2a2ea5a3-6605-4888-bae5-df756037ea07"
-          (reference "#PWR084") (unit 1)
+          (reference "#PWR063") (unit 1)
         )
       )
@@
   (symbol (lib_id "power:VDD") (at 83.82 88.9 0) (unit 1)
     (in_bom yes) (on_board yes) (dnp no) (fields_autoplaced)
-    (property "Reference" "#PWR078" (at 83.82 92.71 0)
+    (property "Reference" "#PWR057" (at 83.82 92.71 0)
       (effects (font (size 1.27 1.27)) hide)
     )
@@
       (project "watch"
         (path "/7f737de8-b7e5-4967-9e9f-b541c91fc2b3/2a2ea5a3-6605-4888-bae5-df756037ea07"
-          (reference "#PWR078") (unit 1)
-        )
-      )
+          (reference "#PWR057") (unit 1)
+        )
+      )

Commit message: Routing progress
Parts:
- removed C26: 0.1u, Capacitor_SMD:C_0402_1005Metric_Pad0.74x0.62mm_HandSolder, symbol Device:C_Small
Connections:
- net DISP_ON is gone; now on net VDD: DS1.5 (DISP)
- net INVERT is gone; now on net GND: DS1.4 (EXTCOMIN)
- net GND: now also DS1.8 (EXTMODE)
- net VDD: no longer DS1.3 (SCS)
- new net DISP_CS: DS1.3 (SCS)
Changed lines of the file:
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@@
 (kicad_sch (version 20230121) (generator eeschema)
   (paper "A4")
-  (junction (at 83.82 97.79) (diameter 0) (color 0 0 0 0)
-  )
-  (wire (pts (xy 81.28 97.79) (xy 83.82 97.79))
-    (stroke (width 0) (type default))
-  )
-  (wire (pts (xy 83.82 104.14) (xy 83.82 105.41))
+  (junction (at 95.25 107.95) (diameter 0) (color 0 0 0 0)
+  )
+  (wire (pts (xy 95.25 109.22) (xy 95.25 107.95))
+    (stroke (width 0) (type default))
+  )
+  (wire (pts (xy 95.25 104.14) (xy 95.25 107.95))
     (stroke (width 0) (type default))
   )
@@
     (stroke (width 0) (type default))
   )
-  (wire (pts (xy 83.82 97.79) (xy 83.82 99.06))
+  (wire (pts (xy 96.52 104.14) (xy 95.25 104.14))
     (stroke (width 0) (type default))
   )
@@
     (stroke (width 0) (type default))
   )
-  (wire (pts (xy 83.82 97.79) (xy 96.52 97.79))
+  (wire (pts (xy 95.25 107.95) (xy 96.52 107.95))
     (stroke (width 0) (type default))
   )
@@
     (stroke (width 0) (type default))
   )
-  (wire (pts (xy 96.52 91.44) (xy 83.82 91.44))
-    (stroke (width 0) (type default))
-  )
   (wire (pts (xy 157.48 93.98) (xy 157.48 95.25))
     (stroke (width 0) (type default))
   )
-  (wire (pts (xy 83.82 91.44) (xy 83.82 88.9))
+  (wire (pts (xy 96.52 97.79) (xy 80.01 97.79))
+    (stroke (width 0) (type default))
+  )
+  (wire (pts (xy 80.01 93.98) (xy 80.01 97.79))
     (stroke (width 0) (type default))
   )
@@
     (effects (font (size 1.27 1.27)) (justify right))
   )
-  (hierarchical_label "DISP_ON" (shape input) (at 81.28 97.79 180) (fields_autoplaced)
-    (effects (font (size 1.27 1.27)) (justify right))
-  )
   (hierarchical_label "SDI" (shape input) (at 96.52 87.63 180) (fields_autoplaced)
     (effects (font (size 1.27 1.27)) (justify right))
   )
-  (hierarchical_label "INVERT" (shape input) (at 96.52 104.14 180) (fields_autoplaced)
+  (hierarchical_label "DISP_CS" (shape input) (at 96.52 91.44 180) (fields_autoplaced)
     (effects (font (size 1.27 1.27)) (justify right))
   )
@@
     )
   )
+  (symbol (lib_id "power:GND") (at 95.25 109.22 0) (unit 1)
+    (in_bom yes) (on_board yes) (dnp no) (fields_autoplaced)
+    (property "Reference" "#PWR04" (at 95.25 115.57 0)
+      (effects (font (size 1.27 1.27)) hide)
+    )
+    (property "Value" "GND" (at 95.25 114.3 0)
+      (effects (font (size 1.27 1.27)))
+    )
+    (property "Footprint" "" (at 95.25 109.22 0)
+      (effects (font (size 1.27 1.27)) hide)
+    )
+    (property "Datasheet" "" (at 95.25 109.22 0)
+      (effects (font (size 1.27 1.27)) hide)
+    )
+    (pin "1")
+    (instances
+      (project "watch"
+        (path "/7f737de8-b7e5-4967-9e9f-b541c91fc2b3/2a2ea5a3-6605-4888-bae5-df756037ea07"
+          (reference "#PWR04") (unit 1)
+        )
+      )
+    )
+  )
   (symbol (lib_id "power:VDD") (at 157.48 93.98 0) (unit 1)
     (in_bom yes) (on_board yes) (dnp no) (fields_autoplaced)
@@
         (path "/7f737de8-b7e5-4967-9e9f-b541c91fc2b3/2a2ea5a3-6605-4888-bae5-df756037ea07"
           (reference "#PWR058") (unit 1)
-        )
-      )
-    )
-  )
-  (symbol (lib_id "power:GND") (at 83.82 105.41 0) (unit 1)
-    (in_bom yes) (on_board yes) (dnp no) (fields_autoplaced)
-    (property "Reference" "#PWR062" (at 83.82 111.76 0)
-      (effects (font (size 1.27 1.27)) hide)
-    )
-    (property "Value" "GND" (at 83.82 110.49 0)
-      (effects (font (size 1.27 1.27)))
-    )
-    (property "Footprint" "" (at 83.82 105.41 0)
-      (effects (font (size 1.27 1.27)) hide)
-    )
-    (property "Datasheet" "" (at 83.82 105.41 0)
-      (effects (font (size 1.27 1.27)) hide)
-    )
-    (pin "1")
-    (instances
-      (project "watch"
-        (path "/7f737de8-b7e5-4967-9e9f-b541c91fc2b3/2a2ea5a3-6605-4888-bae5-df756037ea07"
-          (reference "#PWR062") (unit 1)
-        )
-      )
-    )
-  )
-  (symbol (lib_id "Device:C_Small") (at 83.82 101.6 0) (unit 1)
-    (in_bom yes) (on_board yes) (dnp no)
-    (property "Reference" "C26" (at 81.28 100.33 0)
-      (effects (font (size 1.27 1.27)) (justify right))
-    )
-    (property "Value" "0.1u" (at 81.28 102.87 0)
-      (effects (font (size 1.27 1.27)) (justify right))
-    )
-    (property "Footprint" "Capacitor_SMD:C_0402_1005Metric_Pad0.74x0.62mm_HandSolder" (at 83.82 101.6 0)
-      (effects (font (size 1.27 1.27)) hide)
-    )
-    (property "Datasheet" "~" (at 83.82 101.6 0)
-      (effects (font (size 1.27 1.27)) hide)
-    )
-    (pin "1")
-    (pin "2")
-    (instances
-      (project "watch"
-        (path "/7f737de8-b7e5-4967-9e9f-b541c91fc2b3/2a2ea5a3-6605-4888-bae5-df756037ea07"
-          (reference "C26") (unit 1)
         )
       )
@@
     )
   )
-  (symbol (lib_id "power:VDD") (at 83.82 88.9 0) (unit 1)
-    (in_bom yes) (on_board yes) (dnp no) (fields_autoplaced)
-    (property "Reference" "#PWR057" (at 83.82 92.71 0)
-      (effects (font (size 1.27 1.27)) hide)
-    )
-    (property "Value" "VDD" (at 83.82 83.82 0)
-      (effects (font (size 1.27 1.27)))
-    )
-    (property "Footprint" "" (at 83.82 88.9 0)
-      (effects (font (size 1.27 1.27)) hide)
-    )
-    (property "Datasheet" "" (at 83.82 88.9 0)
-      (effects (font (size 1.27 1.27)) hide)
-    )
+  (symbol (lib_id "power:VDD") (at 80.01 93.98 0) (unit 1)
+    (in_bom yes) (on_board yes) (dnp no) (fields_autoplaced)
+    (property "Reference" "#PWR057" (at 80.01 97.79 0)
+      (effects (font (size 1.27 1.27)) hide)
+    )
+    (property "Value" "VDD" (at 80.01 88.9 0)
+      (effects (font (size 1.27 1.27)))
+    )
+    (property "Footprint" "" (at 80.01 93.98 0)
+      (effects (font (size 1.27 1.27)) hide)
+    )
+    (property "Datasheet" "" (at 80.01 93.98 0)
+      (effects (font (size 1.27 1.27)) hide)
+    )

Commit message: Clean up library symbols, update to kicad 8
Parts:
- C24, C25: value 1u -> 1uF

Commit message: Add manufacturer/PN fields, select LCSC parts
Parts:
- C24, C25: LCSC (none) -> C52923
- DS1: LCSC (none) -> C5591388
Changed lines of the file:
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@@
+			)
+		)
+		(property "LCSC" "C5591388"
+			(at 111.76 96.52 0)
+			(effects
+				(font
+					(size 1.27 1.27)
+				)
+				(hide yes)
 			)
 		)
@@
 			)
 		)
+		(property "LCSC" "C52923"
+			(at 157.48 97.79 0)
+			(effects
+				(font
+					(size 1.27 1.27)
+				)
+				(hide yes)
+			)
+		)
 		(pin "1"
 		)
@@
 			(at 170.18 97.79 0)
 			(effects
+				(font
+					(size 1.27 1.27)
+				)
+				(hide yes)
+			)
+		)
+		(property "LCSC" "C52923"
+			(at 170.18 97.79 0)
+			(effects

Commit message: Finish adding MPN info
Parts:
- C24, C25: Manufacturer (none) -> Samsung; Manufacturer Part Number (none) -> CL05A105KA5NQNC
- DS1: LCSC C5591388 -> (none); Manufacturer (none) -> Panasonic; Manufacturer Part Number (none) -> AYF531035A
Changed lines of the file:
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@@
 			)
 		)
-		(property "LCSC" "C5591388"
+		(property "LCSC" ""
+			(at 111.76 96.52 0)
+			(effects
+				(font
+					(size 1.27 1.27)
+				)
+				(hide yes)
+			)
+		)
+		(property "Manufacturer" "Panasonic"
+			(at 111.76 96.52 0)
+			(effects
+				(font
+					(size 1.27 1.27)
+				)
+				(hide yes)
+			)
+		)
+		(property "Manufacturer Part Number" "AYF531035A"
 			(at 111.76 96.52 0)
 			(effects
@@
 			)
 		)
+		(property "Manufacturer" "Samsung"
+			(at 157.48 97.79 0)
+			(effects
+				(font
+					(size 1.27 1.27)
+				)
+				(hide yes)
+			)
+		)
+		(property "Manufacturer Part Number" "CL05A105KA5NQNC"
+			(at 157.48 97.79 0)
+			(effects
+				(font
+					(size 1.27 1.27)
+				)
+				(hide yes)
+			)
+		)
 		(pin "1"
 		)
@@
 			(at 170.18 97.79 0)
 			(effects
+				(font
+					(size 1.27 1.27)
+				)
+				(hide yes)
+			)
+		)
+		(property "Manufacturer" "Samsung"
+			(at 170.18 97.79 0)
+			(effects
+				(font
+					(size 1.27 1.27)
+				)
+				(hide yes)
+			)
+		)
+		(property "Manufacturer Part Number" "CL05A105KA5NQNC"
+			(at 170.18 97.79 0)
+			(effects
