File: watch_hw/soc.kicad_sch (KiCad schematic)
At the start: 23 parts, among them J3 Conn_ARM_SWD_TagConnect_TC203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, U1 STM32WB55CGUx, X1 NX2016SA-32M, X2 NX2012_32K768

Commit message: Add manufacturer/PN fields, select LCSC parts
Parts:
- C1, C10, C12, C3, C4, C5: LCSC (none) -> C1525
- C11, C9: LCSC (none) -> C19666
- C13, C14: LCSC (none) -> C32949
- C2: LCSC (none) -> C26409
- C6: LCSC (none) -> C23733
- C7: LCSC (none) -> C15195
- C8: LCSC (none) -> C52923
- R1, R2: LCSC (none) -> C25744
- R3, R4: LCSC (none) -> C25900
- U1: LCSC (none) -> C404023
- X1: LCSC (none) -> C843260
- X2: LCSC (none) -> C891748
Changed lines of the file:
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@@
 			)
 		)
+		(property "LCSC" "C19666"
+			(at 38.1 133.35 0)
+			(effects
+				(font
+					(size 1.27 1.27)
+				)
+				(hide yes)
+			)
+		)
 		(pin "2"
 		)
@@
 			)
 		)
+		(property "LCSC" "C26409"
+			(at 50.8 158.75 0)
+			(effects
+				(font
+					(size 1.27 1.27)
+				)
+				(hide yes)
+			)
+		)
 		(pin "2"
 		)
@@
 			)
 		)
+		(property "LCSC" "C52923"
+			(at 139.7 158.75 0)
+			(effects
+				(font
+					(size 1.27 1.27)
+				)
+				(hide yes)
+			)
+		)
 		(pin "2"
 		)
@@
 			)
 		)
+		(property "LCSC" "C1525"
+			(at 71.12 158.75 0)
+			(effects
+				(font
+					(size 1.27 1.27)
+				)
+				(hide yes)
+			)
+		)
 		(pin "2"
 		)
@@
 			)
 		)
+		(property "LCSC" "C891748"
+			(at 241.3 135.89 0)
+			(effects
+				(font
+					(size 1.27 1.27)
+				)
+				(hide yes)
+			)
+		)
 		(pin "2"
 		)
@@
 			)
 		)
+		(property "LCSC" "C25900"
+			(at 175.26 109.22 0)
+			(effects
+				(font
+					(size 1.27 1.27)
+				)
+				(hide yes)
+			)
+		)
 		(pin "1"
 		)
@@
 			)
 		)
+		(property "LCSC" "C1525"
+			(at 38.1 158.75 0)
+			(effects
+				(font
+					(size 1.27 1.27)
+				)
+				(hide yes)
+			)
+		)
 		(pin "2"
 		)
@@
 			)
 		)
+		(property "LCSC" "C15195"
+			(at 127 158.75 0)
+			(effects
+				(font
+					(size 1.27 1.27)
+				)
+				(hide yes)
+			)
+		)
 		(pin "2"
 		)
@@
 			)
 		)
+		(property "LCSC" "C32949"
+			(at 236.22 139.7 0)
+			(effects
+				(font
+					(size 1.27 1.27)
+				)
+				(hide yes)
+			)
+		)
 		(pin "2"
 		)
@@
 			)
 		)
+		(property "LCSC" "C843260"
+			(at 241.3 110.49 0)
+			(effects
+				(font
+					(size 1.27 1.27)
+				)
+				(hide yes)
+			)
+		)
 		(pin "2"
 		)
@@
 			)
 		)
+		(property "LCSC" "C32949"
+			(at 246.38 139.7 0)
+			(effects
+				(font
+					(size 1.27 1.27)
+				)
+				(hide yes)
+			)
+		)
 		(pin "2"
 		)
@@
 			)
 		)
+		(property "LCSC" "C1525"
+			(at 83.82 158.75 0)
+			(effects
+				(font
+					(size 1.27 1.27)
+				)
+				(hide yes)
+			)
+		)
 		(pin "2"
 		)
@@
 			)
 		)
+		(property "LCSC" "C1525"
+			(at 57.15 59.69 0)
+			(effects
+				(font
+					(size 1.27 1.27)
+				)
+				(hide yes)
+			)
+		)
 		(pin "2"
 		)
@@
 			)
 		)
+		(property "LCSC" "C1525"
+			(at 158.75 158.75 0)
+			(effects
+				(font
+					(size 1.27 1.27)
+				)
+				(hide yes)
+			)
+		)
 		(pin "2"
 		)
@@
 			)
 		)
+		(property "LCSC" "C25744"
+			(at 57.15 52.07 0)
+			(effects
+				(font
+					(size 1.27 1.27)
+				)
+				(hide yes)
+			)
+		)
 		(pin "1"
 		)
@@
 			)
 		)
+		(property "LCSC" "C25744"
+			(at 80.01 87.63 0)
+			(effects
+				(font
+					(size 1.27 1.27)
+				)
+				(hide yes)
+			)
+		)
 		(pin "1"
 		)
@@
 			)
 		)
+		(property "LCSC" "C19666"
+			(at 69.85 80.01 0)
+			(effects
+				(font
+					(size 1.27 1.27)
+				)
+				(hide yes)
+			)
+		)
 		(pin "2"
 		)
@@
 			)
 		)
+		(property "LCSC" "C23733"
+			(at 109.22 158.75 0)
+			(effects
+				(font
+					(size 1.27 1.27)
+				)
+				(hide yes)
+			)
+		)
 		(pin "2"
 		)
@@
 			)
 		)
+		(property "LCSC" "C25900"
+			(at 166.37 109.22 0)
+			(effects
+				(font
+					(size 1.27 1.27)
+				)
+				(hide yes)
+			)
+		)
 		(pin "1"
 		)
@@
 			)
 		)
+		(property "LCSC" "C404023"
+			(at 121.92 88.9 0)
+			(effects
+				(font
+					(size 1.27 1.27)
+				)
+				(hide yes)
+			)
+		)
 		(pin "6"
 		)
@@
 			(at 96.52 158.75 0)
 			(effects
+				(font
+					(size 1.27 1.27)
+				)
+				(hide yes)
+			)
+		)
+		(property "LCSC" "C1525"
+			(at 96.52 158.75 0)
+			(effects

Commit message: Finish adding MPN info
Parts:
- C1, C10, C12, C3, C4, C5: Manufacturer (none) -> Samsung; Manufacturer Part Number (none) -> CL05B104KO5NNNC
- C11, C9: Manufacturer (none) -> Samsung; Manufacturer Part Number (none) -> CL10A475KO8NNNC
- C13, C14: Manufacturer (none) -> Samsung; Manufacturer Part Number (none) -> CL05C100JB5NNNC
- C2: Manufacturer (none) -> Samsung; Manufacturer Part Number (none) -> CL05C101JB5NNNC
- C6: Manufacturer (none) -> Samsung; Manufacturer Part Number (none) -> CL05A475MP5NRNC
- C7: Manufacturer (none) -> Samsung; Manufacturer Part Number (none) -> CL05B103KB5NNNC
- C8: Manufacturer (none) -> Samsung; Manufacturer Part Number (none) -> CL05A105KA5NQNC
- L1: LCSC (none) -> C162582; Manufacturer Part Number LQM21FN100M70L -> LQM21FN100M80L
- R1, R2: Manufacturer (none) -> UNI-ROYAL; Manufacturer Part Number (none) -> 0402WGF1002TCE
- R3, R4: Manufacturer (none) -> UNI-ROYAL; Manufacturer Part Number (none) -> 0402WGF4701TCE
- U1: Manufacturer (none) -> ST; Manufacturer Part Number (none) -> STM32WB55CGU6
- X1: Manufacturer (none) -> NDK; Manufacturer Part Number (none) -> NX2016SA-32MHZ-STD-CZS-5
- X2: Manufacturer (none) -> NDK; Manufacturer Part Number (none) -> NX2012SA-32.768KHZ-STD-MUB-2
