File: watch_hw/watch.kicad_sch (KiCad schematic)
At the start: 7 parts, among them J1 USB_B_Micro, SW1 TL6340AF160Q, SW2 TL6340AF160Q

Commit message: Finish adding MPN info
Parts:
- J1: value USB_B_Micro -> UJ2-MIBH-4-SMT-TR-67; Manufacturer (none) -> CUI; Manufacturer Part Number (none) -> UJ2-MIBH-4-SMT-TR-67
- R7, R8: Manufacturer (none) -> UNI-ROYAL; Manufacturer Part Number (none) -> 0402WGF1002TCE
- SW1, SW2: Manufacturer (none) -> E-Switch; Manufacturer Part Number (none) -> TL6340AF160Q
Changed lines of the file:
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@@
+			)
+		)
+		(property "Manufacturer" "UNI-ROYAL"
+			(at 223.52 118.11 0)
+			(effects
+				(font
+					(size 1.27 1.27)
+				)
+				(hide yes)
+			)
+		)
+		(property "Manufacturer Part Number" "0402WGF1002TCE"
+			(at 223.52 118.11 0)
+			(effects
+				(font
+					(size 1.27 1.27)
+				)
+				(hide yes)
 			)
 		)
@@
 			)
 		)
+		(property "Manufacturer" "E-Switch"
+			(at 198.12 128.27 90)
+			(effects
+				(font
+					(size 1.27 1.27)
+				)
+				(hide yes)
+			)
+		)
+		(property "Manufacturer Part Number" "TL6340AF160Q"
+			(at 198.12 128.27 90)
+			(effects
+				(font
+					(size 1.27 1.27)
+				)
+				(hide yes)
+			)
+		)
 		(pin "1"
 		)
@@
 			)
 		)
+		(property "Manufacturer" "E-Switch"
+			(at 223.52 128.27 90)
+			(effects
+				(font
+					(size 1.27 1.27)
+				)
+				(hide yes)
+			)
+		)
+		(property "Manufacturer Part Number" "TL6340AF160Q"
+			(at 223.52 128.27 90)
+			(effects
+				(font
+					(size 1.27 1.27)
+				)
+				(hide yes)
+			)
+		)
 		(pin "1"
 		)
@@
 			)
 		)
+		(property "Manufacturer" "UNI-ROYAL"
+			(at 198.12 118.11 0)
+			(effects
+				(font
+					(size 1.27 1.27)
+				)
+				(hide yes)
+			)
+		)
+		(property "Manufacturer Part Number" "0402WGF1002TCE"
+			(at 198.12 118.11 0)
+			(effects
+				(font
+					(size 1.27 1.27)
+				)
+				(hide yes)
+			)
+		)
 		(pin "1"
 		)
@@
 			)
 		)
-		(property "Value" "USB_B_Micro"
+		(property "Value" "UJ2-MIBH-4-SMT-TR-67"
 			(at 187.96 59.69 0)
 			(effects
@@
 			(at 187.96 69.85 0)
 			(effects
+				(font
+					(size 1.27 1.27)
+				)
+				(hide yes)
+			)
+		)
+		(property "Manufacturer" "CUI"
+			(at 187.96 69.85 0)
+			(effects
+				(font
+					(size 1.27 1.27)
+				)
+				(hide yes)
+			)
+		)
+		(property "Manufacturer Part Number" "UJ2-MIBH-4-SMT-TR-67"
+			(at 187.96 69.85 0)
+			(effects
